File: hw/stm8-kid-toy.sch (KiCad schematic (older format))
At the start: 14 parts, among them SW1 SW_Push, SW2 SW_Push, SW3 SW_Push, U1 STM8S003F3P

Commit message: fix sch again
Parts:
- removed D?: DIODE, symbol Simulation_SPICE:DIODE
- added D? (x3): DIODE, symbol Simulation_SPICE:DIODE
Connections:
- net BTN1: now also D?.2 (K); no longer R?.1, SW1.2
- net BTN2: now also D?.2 (K); no longer R?.1, SW2.2
- net BTN3: now also D?.2 (K); no longer R?.1, SW3.2
- net COM1: now also SW1.1, SW2.1, SW3.1
- new net: R?.1, SW1.2
- new net: D?.1 (A), R?.1, SW2.2
- new net: D?.1 (A), R?.1, SW3.2
Other:
- moved on the sheet: R?, SW1, SW2, SW3
Changed lines of the file:
@@
 	2850 2800 2850 1800
 Wire Wire Line
-	3525 1400 3525 1500
-Wire Wire Line
-	3525 1400 4075 1400
-Wire Wire Line
-	4075 1400 4075 1500
-Wire Wire Line
-	4075 1400 4625 1400
-Wire Wire Line
-	4625 1400 4625 1500
-Connection ~ 4075 1400
+	4125 1400 4125 1500
+Wire Wire Line
+	4475 1400 4475 1500
+Wire Wire Line
+	4475 1400 4825 1400
+Wire Wire Line
+	4825 1400 4825 1500
+Connection ~ 4475 1400
 $Comp
 L Device:LED D1
@@
 L Switch:SW_Push SW1
 U 1 1 5D99E0C8
-P 3525 1700
-F 0 "SW1" V 3479 1848 50  0000 L CNN
-F 1 "SW_Push" V 3570 1848 50  0000 L CNN
-F 2 "" H 3525 1900 50  0001 C CNN
-F 3 "~" H 3525 1900 50  0001 C CNN
-	1    3525 1700
+P 4125 1700
+F 0 "SW1" V 4079 1848 50  0000 L CNN
+F 1 "SW_Push" V 4170 1848 50  0001 L CNN
+F 2 "" H 4125 1900 50  0001 C CNN
+F 3 "~" H 4125 1900 50  0001 C CNN
+	1    4125 1700
 	0    1    1    0
 $EndComp
@@
 L Switch:SW_Push SW2
 U 1 1 5D99E652
-P 4075 1700
-F 0 "SW2" V 4029 1848 50  0000 L CNN
-F 1 "SW_Push" V 4120 1848 50  0000 L CNN
-F 2 "" H 4075 1900 50  0001 C CNN
-F 3 "~" H 4075 1900 50  0001 C CNN
-	1    4075 1700
+P 4475 1700
+F 0 "SW2" V 4429 1848 50  0000 L CNN
+F 1 "SW_Push" V 4520 1848 50  0001 L CNN
+F 2 "" H 4475 1900 50  0001 C CNN
+F 3 "~" H 4475 1900 50  0001 C CNN
+	1    4475 1700
 	0    1    1    0
 $EndComp
@@
 L Switch:SW_Push SW3
 U 1 1 5D99ED0D
-P 4625 1700
-F 0 "SW3" V 4579 1848 50  0000 L CNN
-F 1 "SW_Push" V 4670 1848 50  0000 L CNN
-F 2 "" H 4625 1900 50  0001 C CNN
-F 3 "~" H 4625 1900 50  0001 C CNN
-	1    4625 1700
+P 4825 1700
+F 0 "SW3" V 4779 1848 50  0000 L CNN
+F 1 "SW_Push" V 4870 1848 50  0001 L CNN
+F 2 "" H 4825 1900 50  0001 C CNN
+F 3 "~" H 4825 1900 50  0001 C CNN
+	1    4825 1700
 	0    1    1    0
 $EndComp
@@
 Text GLabel 1575 2325 0    50   Input ~ 0
 LED1
-Wire Wire Line
-	2500 1400 2850 1400
-Text GLabel 3250 2000 0    50   Input ~ 0
+Text GLabel 3325 2000 0    50   Input ~ 0
 BTN1
-Text GLabel 3250 2175 0    50   Input ~ 0
+Text GLabel 3325 2175 0    50   Input ~ 0
 BTN2
-Text GLabel 3250 2350 0    50   Input ~ 0
+Text GLabel 3325 2350 0    50   Input ~ 0
 BTN3
 Wire Wire Line
-	3250 2000 3525 2000
-Wire Wire Line
-	3250 2175 4075 2175
-Wire Wire Line
-	3250 2350 4625 2350
-$Comp
-L Simulation_SPICE:DIODE D?
-U 1 1 5DA61785
-P 3250 1400
-F 0 "D?" V 3204 1480 50  0000 L CNN
-F 1 "DIODE" V 3295 1480 50  0000 L CNN
-F 2 "" H 3250 1400 50  0001 C CNN
-F 3 "~" H 3250 1400 50  0001 C CNN
-F 4 "Y" H 3250 1400 50  0001 L CNN "Spice_Netlist_Enabled"
-F 5 "V" H 3250 1400 50  0001 L CNN "Spice_Primitive"
-	1    3250 1400
-	1    0    0    -1
-$EndComp
-Wire Wire Line
-	2850 1400 3100 1400
-Connection ~ 2850 1400
-Wire Wire Line
-	3400 1400 3525 1400
-Connection ~ 3525 1400
+	3325 2000 3500 2000
+Wire Wire Line
+	3325 2175 3500 2175
+Wire Wire Line
+	3325 2350 3500 2350
+Connection ~ 4125 1400
 $Comp
 L Device:R R?
@@
 L Device:R R?
 U 1 1 5DA74885
-P 4075 2600
-F 0 "R?" H 4145 2646 50  0000 L CNN
-F 1 "R" H 4145 2555 50  0000 L CNN
-F 2 "" V 4005 2600 50  0001 C CNN
-F 3 "~" H 4075 2600 50  0001 C CNN
-	1    4075 2600
+P 4475 2600
+F 0 "R?" H 4545 2646 50  0000 L CNN
+F 1 "R" H 4545 2555 50  0000 L CNN
+F 2 "" V 4405 2600 50  0001 C CNN
+F 3 "~" H 4475 2600 50  0001 C CNN
+	1    4475 2600
 	1    0    0    -1
 $EndComp
@@
 L Device:R R?
 U 1 1 5DA74D1A
-P 4625 2600
-F 0 "R?" H 4695 2646 50  0000 L CNN
-F 1 "R" H 4695 2555 50  0000 L CNN
-F 2 "" V 4555 2600 50  0001 C CNN
-F 3 "~" H 4625 2600 50  0001 C CNN
-	1    4625 2600
+P 4825 2600
+F 0 "R?" H 4895 2646 50  0000 L CNN
+F 1 "R" H 4895 2555 50  0000 L CNN
+F 2 "" V 4755 2600 50  0001 C CNN
+F 3 "~" H 4825 2600 50  0001 C CNN
+	1    4825 2600
 	1    0    0    -1
 $EndComp
-Text GLabel 3250 2800 0    50   Input ~ 0
+Text GLabel 3325 2800 0    50   Input ~ 0
 GND
 $Comp
 L Device:R R?
 U 1 1 5DA73BCF
-P 3525 2600
-F 0 "R?" H 3595 2646 50  0000 L CNN
-F 1 "R" H 3595 2555 50  0000 L CNN
-F 2 "" V 3455 2600 50  0001 C CNN
-F 3 "~" H 3525 2600 50  0001 C CNN
-	1    3525 2600
+P 4125 2600
+F 0 "R?" H 4195 2646 50  0000 L CNN
+F 1 "R" H 4195 2555 50  0000 L CNN
+F 2 "" V 4055 2600 50  0001 C CNN
+F 3 "~" H 4125 2600 50  0001 C CNN
+	1    4125 2600
 	1    0    0    -1
 $EndComp
 Wire Wire Line
-	3525 1900 3525 2000
-Wire Wire Line
-	4075 1900 4075 2175
-Wire Wire Line
-	4625 1900 4625 2350
-Wire Wire Line
-	3525 2000 3525 2450
-Connection ~ 3525 2000
-Wire Wire Line
-	4075 2175 4075 2450
-Connection ~ 4075 2175
-Wire Wire Line
-	4625 2350 4625 2450
-Connection ~ 4625 2350
-Wire Wire Line
-	4625 2750 4625 2800
-Wire Wire Line
-	4625 2800 4075 2800
-Wire Wire Line
-	3525 2750 3525 2800
-Connection ~ 3525 2800
-Wire Wire Line
-	3525 2800 3250 2800
-Wire Wire Line
-	4075 2750 4075 2800
-Connection ~ 4075 2800
-Wire Wire Line
-	4075 2800 3525 2800
+	4825 2750 4825 2800
+Wire Wire Line
+	4125 2750 4125 2800
+Wire Wire Line
+	4475 2750 4475 2800
+Connection ~ 4475 2800
 Text GLabel 1750 1600 0    50   Input ~ 0
 COM2
 Text GLabel 1750 1800 0    50   Input ~ 0
 COM3
+$Comp
+L Simulation_SPICE:DIODE D?
+U 1 1 5DBA5698
+P 3650 2000
+F 0 "D?" V 3475 1900 50  0000 L CNN
+F 1 "DIODE" V 3695 2080 50  0001 L CNN
+F 2 "" H 3650 2000 50  0001 C CNN
+F 3 "~" H 3650 2000 50  0001 C CNN
+F 4 "Y" H 3650 2000 50  0001 L CNN "Spice_Netlist_Enabled"
+F 5 "V" H 3650 2000 50  0001 L CNN "Spice_Primitive"
+	1    3650 2000
+	-1   0    0    1
+$EndComp
+$Comp
+L Simulation_SPICE:DIODE D?
+U 1 1 5DBA725E
+P 3650 2350
+F 0 "D?" V 3475 2250 50  0000 L CNN
+F 1 "DIODE" V 3695 2430 50  0001 L CNN
+F 2 "" H 3650 2350 50  0001 C CNN
+F 3 "~" H 3650 2350 50  0001 C CNN
+F 4 "Y" H 3650 2350 50  0001 L CNN "Spice_Netlist_Enabled"
+F 5 "V" H 3650 2350 50  0001 L CNN "Spice_Primitive"
+	1    3650 2350
+	-1   0    0    1
+$EndComp
+Wire Wire Line
+	4125 1900 4125 2000
+Wire Wire Line
+	4475 1900 4475 2175
+Wire Wire Line
+	4825 1900 4825 2350
+$Comp
+L Simulation_SPICE:DIODE D?
+U 1 1 5DBA6853
+P 3650 2175
+F 0 "D?" V 3475 2075 50  0000 L CNN
+F 1 "DIODE" V 3695 2255 50  0001 L CNN
+F 2 "" H 3650 2175 50  0001 C CNN
+F 3 "~" H 3650 2175 50  0001 C CNN
+F 4 "Y" H 3650 2175 50  0001 L CNN "Spice_Netlist_Enabled"
+F 5 "V" H 3650 2175 50  0001 L CNN "Spice_Primitive"
+	1    3650 2175
+	-1   0    0    1
+$EndComp
+Wire Wire Line
+	3825 2000 4125 2000
+Connection ~ 4125 2000
+Wire Wire Line
+	4125 2000 4125 2450
+Wire Wire Line
+	4125 1400 4475 1400
+Wire Wire Line
+	4825 2800 4475 2800
+Wire Wire Line
+	2500 1400 2850 1400
+Wire Wire Line
+	2850 1400 4125 1400
+Connection ~ 2850 1400
+Wire Wire Line
+	3800 2175 4475 2175
+Connection ~ 4475 2175
+Wire Wire Line
+	4475 2175 4475 2450
+Wire Wire Line
+	3800 2350 4825 2350
+Connection ~ 4825 2350
+Wire Wire Line
+	4825 2350 4825 2450
+Wire Wire Line
+	3325 2800 4125 2800
+Connection ~ 4125 2800
+Wire Wire Line
+	4125 2800 4475 2800
 $EndSCHEMATC
